File: pcb/model-b/model-b.kicad_sch (KiCad schematic)
At the start: 208 parts, among them SW1 SW_ESC, SW10 SW_F9, SW11 SW_F10, SW12 SW_F11, SW13 SW_F12, SW14 SW_`~, SW15 SW_1, SW16 SW_2, SW17 SW_3, SW18 SW_4, SW19 SW_5, SW2 SW_F1, SW20 SW_6, SW21 SW_7, SW22 SW_8, SW23 SW_9, SW24 SW_0, SW25 SW_-, SW26 SW_=, SW27 SW_BACKSPACE, SW28 SW_TAB, SW29 SW_Q, SW3 SW_F2, SW30 SW_W, SW31 SW_E, SW32 SW_R, SW33 SW_T, SW34 SW_Y, SW35 SW_U, SW36 SW_I, SW37 SW_O, SW38 SW_P, SW39 SW_[, SW4 SW_F3, SW40 SW_], SW41 SW_\, SW42 SW_CAPS, SW43 SW_A, SW44 SW_S, SW45 SW_D, SW46 SW_F, SW47 SW_G, SW48 SW_H, SW49 SW_J, SW5 SW_F4, SW50 SW_K, SW51 SW_L, SW52 SW_;, SW53 SW_', SW55 SW_ENTER, SW56 SW_LSHIFT, SW57 SW_Z, SW58 SW_X, SW59 SW_C, SW6 SW_F5, SW60 SW_V, SW61 SW_B, SW62 SW_N, SW63 SW_M, SW64 SW_,, SW65 SW_., SW66 SW_/, SW68 SW_RSHIFT, SW69 SW_UP, SW7 SW_F6, SW70 SW_LCTRL, SW71 SW_LWIN, SW72 SW_LALT, SW73 SW_SPACE, SW74 SW_RALT, SW75 SW_FN, SW76 SW_RCTRL, SW77 SW_LEFT, SW78 SW_DOWN, SW8 SW_F7, SW80 SW_DEL, SW81 SW_INSERT, SW82 SW_HOME, SW83 SW_END, SW84 SW_RIGHT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

Commit message: finished pcb (probably)
Parts:
- added D67: D, Diode_SMD:D_0402_1005Metric, symbol Device:D
- added SW54: SW_F13, MX_Only:MXOnly-1U-Hotswap, symbol Switch:SW_SPST
Connections:
- net VCC is gone; now on net +3V3: R1.2, R2.2
- net col12: now also SW54.2 (B)
- net row3: now also D67.1 (K)
- new net: D67.2 (A), SW54.1 (A)
Changed lines of the file:
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@@
   (junction (at 190.5 105.41) (diameter 0) (color 0 0 0 0)
   )
+  (junction (at 62.23 147.32) (diameter 0) (color 0 0 0 0)
+  )
   (junction (at 231.14 52.07) (diameter 0) (color 0 0 0 0)
   )
@@
   (junction (at 63.5 97.79) (diameter 0) (color 0 0 0 0)
   )
+  (junction (at 231.14 82.55) (diameter 0) (color 0 0 0 0)
+  )
   (junction (at 190.5 154.94) (diameter 0) (color 0 0 0 0)
   )
@@
   (junction (at 261.62 67.31) (diameter 0) (color 0 0 0 0)
   )
-  (junction (at 62.23 147.32) (diameter 0) (color 0 0 0 0)
-  )
   (junction (at 200.66 82.55) (diameter 0) (color 0 0 0 0)
   )
   (junction (at 48.26 82.55) (diameter 0) (color 0 0 0 0)
   )
+  (junction (at 220.98 90.17) (diameter 0) (color 0 0 0 0)
+  )
   (junction (at 215.9 67.31) (diameter 0) (color 0 0 0 0)
   )
@@
     (stroke (width 0) (type default))
   )
-  (wire (pts (xy 62.23 147.32) (xy 63.5 147.32))
-    (stroke (width 0) (type default))
-  )
   (wire (pts (xy 68.58 105.41) (xy 83.82 105.41))
     (stroke (width 0) (type default))
@@
     (stroke (width 0) (type default))
   )
+  (wire (pts (xy 62.23 147.32) (xy 63.5 147.32))
+    (stroke (width 0) (type default))
+  )
   (wire (pts (xy 39.37 171.45) (xy 39.37 172.72))
     (stroke (width 0) (type default))
@@
     (stroke (width 0) (type default))
   )
+  (wire (pts (xy 220.98 90.17) (xy 236.22 90.17))
+    (stroke (width 0) (type default))
+  )
   (wire (pts (xy 114.3 59.69) (xy 129.54 59.69))
     (stroke (width 0) (type default))
@@
     (stroke (width 0) (type default))
   )
-  (wire (pts (xy 205.74 90.17) (xy 236.22 90.17))
+  (wire (pts (xy 205.74 90.17) (xy 220.98 90.17))
     (stroke (width 0) (type default))
   )
@@
     (stroke (width 0) (type default))
   )
-  (wire (pts (xy 231.14 67.31) (xy 231.14 97.79))
+  (wire (pts (xy 231.14 67.31) (xy 231.14 82.55))
     (stroke (width 0) (type default))
   )
@@
     (stroke (width 0) (type default))
   )
+  (wire (pts (xy 231.14 82.55) (xy 231.14 97.79))
+    (stroke (width 0) (type default))
+  )
   (wire (pts (xy 59.69 167.64) (xy 60.96 167.64))
     (stroke (width 0) (type default))
@@
     )
   )
-  (symbol (lib_id "power:VCC") (at 62.23 147.32 180) (unit 1)
-    (in_bom yes) (on_board yes) (dnp no) (fields_autoplaced)
-    (property "Reference" "#PWR02" (at 62.23 143.51 0)
-      (effects (font (size 1.27 1.27)) hide)
-    )
-    (property "Value" "VCC" (at 62.23 152.4 0)
-      (effects (font (size 1.27 1.27)))
-    )
-    (property "Footprint" "" (at 62.23 147.32 0)
-      (effects (font (size 1.27 1.27)) hide)
-    )
-    (property "Datasheet" "" (at 62.23 147.32 0)
-      (effects (font (size 1.27 1.27)) hide)
-    )
-    (pin "1")
-    (instances
-      (project "model-b"
-        (path "/0538c578-a42e-4bd9-8a80-f7f3c5225a8a"
-          (reference "#PWR02") (unit 1)
-        )
-      )
-      (project "Model K Pico-0.2"
-        (path "/1578113e-a709-4724-a2c3-24a8ca825a3f"
-          (reference "#PWR0101") (unit 1)
-        )
-      )
-    )
-  )
   (symbol (lib_id "Switch:SW_SPST") (at 119.38 67.31 0) (unit 1)
     (in_bom yes) (on_board yes) (dnp no)
@@
     )
   )
+  (symbol (lib_id "Switch:SW_SPST") (at 226.06 82.55 0) (unit 1)
+    (in_bom yes) (on_board yes) (dnp no)
+    (property "Reference" "SW54" (at 226.06 77.47 0)
+      (effects (font (size 1.27 1.27)))
+    )
+    (property "Value" "SW_F13" (at 226.06 80.01 0)
+      (effects (font (size 1.27 1.27)))
+    )
+    (property "Footprint" "MX_Only:MXOnly-1U-Hotswap" (at 226.06 82.55 0)
+      (effects (font (size 1.27 1.27)) hide)
+    )
+    (property "Datasheet" "~" (at 226.06 82.55 0)
+      (effects (font (size 1.27 1.27)) hide)
+    )
+    (pin "1")
+    (pin "2")
+    (instances
+      (project "model-b"
+        (path "/0538c578-a42e-4bd9-8a80-f7f3c5225a8a"
+          (reference "SW54") (unit 1)
+        )
+      )
+    )
+  )
   (symbol (lib_id "Device:D") (at 190.5 71.12 90) (unit 1)
     (in_bom yes) (on_board yes) (dnp no)
@@
     )
   )
+  (symbol (lib_id "Device:D") (at 220.98 86.36 90) (unit 1)
+    (in_bom yes) (on_board yes) (dnp no)
+    (property "Reference" "D67" (at 223.52 86.36 90)
+      (effects (font (size 1.27 1.27)))
+    )
+    (property "Value" "D" (at 222.25 88.9 0)
+      (effects (font (size 1.27 1.27)))
+    )
+    (property "Footprint" "Diode_SMD:D_0402_1005Metric" (at 220.98 86.36 0)
+      (effects (font (size 1.27 1.27)) hide)
+    )
+    (property "Datasheet" "~" (at 220.98 86.36 0)
+      (effects (font (size 1.27 1.27)) hide)
+    )
+    (property "Sim.Device" "D" (at 220.98 86.36 0)
+      (effects (font (size 1.27 1.27)) hide)
+    )
+    (property "Sim.Pins" "1=K 2=A" (at 220.98 86.36 0)
+      (effects (font (size 1.27 1.27)) hide)
+    )
+    (pin "1")
+    (pin "2")
+    (instances
+      (project "model-b"
+        (path "/0538c578-a42e-4bd9-8a80-f7f3c5225a8a"
+          (reference "D67") (unit 1)
+        )
+      )
+    )
+  )
   (symbol (lib_id "power:GND") (at 30.48 187.96 0) (unit 1)
     (in_bom yes) (on_board yes) (dnp no) (fields_autoplaced)
@@
         )
       )
+    )
+  )
+  (symbol (lib_id "power:+3V3") (at 62.23 147.32 180) (unit 1)
+    (in_bom yes) (on_board yes) (dnp no) (fields_autoplaced)
+    (property "Reference" "#PWR02" (at 62.23 143.51 0)
+      (effects (font (size 1.27 1.27)) hide)
+    )
+    (property "Value" "+3V3" (at 62.23 152.4 0)
+      (effects (font (size 1.27 1.27)))
+    )
+    (property "Footprint" "" (at 62.23 147.32 0)
+      (effects (font (size 1.27 1.27)) hide)
+    )
+    (property "Datasheet" "" (at 62.23 147.32 0)
+      (effects (font (size 1.27 1.27)) hide)
+    )
+    (pin "1")
+    (instances
+      (project "model-b"
+        (path "/0538c578-a42e-4bd9-8a80-f7f3c5225a8a"
+          (reference "#PWR02") (unit 1)
+        )
+      )
+      (project "pico"
+        (path "/874ed296-eccb-4006-b065-076cf6d81fab"
+          (reference "#PWR029") (unit 1)
+        )
+      )

Commit message: fixed diodes to be SOD-123 and added case files
Parts:
- D1, D10, D11, D12, D13, D14, D15, D16, D17, D18, D19, D2, D20, D21, D22, D23, D24, D25, D26, D27, D28, D29, D3, D30, D31, D32, D33, D34, D35, D36, D37, D38, D39, D4, D40, D41, D42, D43, D44, D45, D46, D47, D48, D49, D5, D50, D51, D52, D53, D55, D56, D57, D58, D59, D6, D60, D61, D62, D63, D64, D65, D66, D67, D68, D69, D7, D70, D71, D72, D73, D74, D75, D76, D77, D78, D79, D8, D80, D81, D82, D83, D84, D9: footprint Diode_SMD:D_0402_1005Metric -> Diode_SMD:D_SOD-123

Commit message: Finished case, minor changes to PCB, laser cutting files prepped
Connections:
- net USB_DM renamed USB_DN
Changed lines of the file:
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@@
     (effects (font (size 1.27 1.27)) (justify right bottom))
   )
-  (label "USB_DM" (at 49.53 237.49 0) (fields_autoplaced)
+  (label "USB_DN" (at 49.53 237.49 0) (fields_autoplaced)
     (effects (font (size 1.27 1.27)) (justify left bottom))
   )
@@
     (effects (font (size 1.27 1.27)) (justify right bottom))
   )
-  (label "USB_DM" (at 251.46 166.37 0) (fields_autoplaced)
+  (label "USB_DN" (at 251.46 166.37 0) (fields_autoplaced)
     (effects (font (size 1.27 1.27)) (justify left bottom))
   )

Commit message: PCBs ordered, pray they come without errors
Parts:
- added TP1, TP2, TP3, TP4, TP5, TP6, TP7, TP8, TP9: TestPoint, libraries:CustomTestPoint, symbol Connector:TestPoint
Connections:
- net +3V3: now also TP9.1
- net GND: now also TP8.1
- net GPIO24: now also TP7.1
- net at U3.24 (SWCLK): now also TP5.1
- net at U3.25 (SWD): now also TP6.1
- net at U3.35 (GPIO23): now also TP1.1
- net at U3.37 (GPIO25): now also TP2.1
- net at U3.40 (GPIO28_ADC2): now also TP3.1
- net at U3.41 (GPIO29_ADC3): now also TP4.1
- no-connect marks 8 -> 2
